File: NeonMatrix.kicad_pcb (KiCad board)
At the start: 2 copper layers, 264 parts, among them U1 74HC595, U2 74HC595, U3 74HC595, U4 74HC595, U5 74HC595, U6 74HC595, U7 74HC595, U8 74HC595

Commit message: First row
Parts:
- NE1, NE10, NE11, NE12, NE13, NE14, NE15, NE16, NE17, NE18, NE19, NE2, NE20, NE21, NE22, NE23, NE24, NE25, NE26, NE27, NE28, NE29, NE3, NE30, NE31, NE32, NE33, NE34, NE35, NE36, NE37, NE38, NE39, NE4, NE40, NE41, NE42, NE43, NE44, NE45, NE46, NE47, NE48, NE49, NE5, NE50, NE51, NE52, NE53, NE54, NE55, NE56, NE57, NE58, NE59, NE6, NE60, NE61, NE62, NE63, NE64, NE7, NE8, NE9: footprint Connector_PinHeader_2.54mm:PinHeader_1x02_P2.54mm_Horizontal -> NeonMatrix_Connector:NeonBulb; moved to B.Cu
- moved U4 597.4 mm to (-309.3, -1.31)
- moved U2 584.6 mm to (-309.3, 28.5)
- moved U6 574.6 mm to (-309.3, 13.6)
- moved R85 543.0 mm to (-278.8, 4.98), turned to 270 degrees
- moved R94 542.8 mm to (-283.6, 17.7), turned to 270 degrees
- moved R86 536.0 mm to (-283.6, 4.26), turned to 270 degrees
- moved NE43 535.9 mm to (-285.3, 4.13)
- moved U8 535.1 mm to (-261.0, -16.2)
- moved R128 529.5 mm to (-262.1, -6.27), turned to 270 degrees
- moved R93 529.4 mm to (-278.8, 18.4), turned to 270 degrees
- moved U3 525.2 mm to (-309.3, -16.2)
- moved R114 524.8 mm to (-262.1, -19.7), turned to 270 degrees
- moved R113 523.7 mm to (-257.2, -19.0), turned to 270 degrees
- moved D64 523.1 mm to (-259.5, -6.33), turned to 180 degrees
- moved D57 521.7 mm to (-259.5, -19.8), turned to 180 degrees
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Connections:
- net Net-(R1-Pad2) renamed /Sheet595Neon/SheetSingleBulb/SIGNAL
- net Net-(R101-Pad2) renamed /sheet5EFAAFC5/sheet5EF2B6E0/SIGNAL
- net Net-(R103-Pad2) renamed /sheet5EFAAFC5/sheet5EF2B77E/SIGNAL
- net Net-(R105-Pad2) renamed /sheet5EFAAFC5/sheet5EF2B800/SIGNAL
- net Net-(R107-Pad2) renamed /sheet5EFAAFC5/sheet5EF2B8A4/SIGNAL
- net Net-(R109-Pad2) renamed /sheet5EFAAFC5/sheet5EF2B938/SIGNAL
- net Net-(R11-Pad2) renamed /Sheet595Neon/sheet5EF2B8A4/SIGNAL
- net Net-(R111-Pad2) renamed /sheet5EFAAFC5/sheet5EF2B9F4/SIGNAL
- net Net-(R113-Pad2) renamed /sheet5EFAAFC6/SheetSingleBulb/SIGNAL
- net Net-(R115-Pad2) renamed /sheet5EFAAFC6/sheet5EF2B64C/SIGNAL
- net Net-(R117-Pad2) renamed /sheet5EFAAFC6/sheet5EF2B6E0/SIGNAL
- net Net-(R119-Pad2) renamed /sheet5EFAAFC6/sheet5EF2B77E/SIGNAL
- net Net-(R121-Pad2) renamed /sheet5EFAAFC6/sheet5EF2B800/SIGNAL
- net Net-(R123-Pad2) renamed /sheet5EFAAFC6/sheet5EF2B8A4/SIGNAL
- net Net-(R125-Pad2) renamed /sheet5EFAAFC6/sheet5EF2B938/SIGNAL
- net Net-(R127-Pad2) renamed /sheet5EFAAFC6/sheet5EF2B9F4/SIGNAL
- net Net-(R13-Pad2) renamed /Sheet595Neon/sheet5EF2B938/SIGNAL
- net Net-(R15-Pad2) renamed /Sheet595Neon/sheet5EF2B9F4/SIGNAL
- net Net-(R17-Pad2) renamed /sheet5EFA929F/SheetSingleBulb/SIGNAL
- net Net-(R19-Pad2) renamed /sheet5EFA929F/sheet5EF2B64C/SIGNAL
- net Net-(R21-Pad2) renamed /sheet5EFA929F/sheet5EF2B6E0/SIGNAL
- net Net-(R23-Pad2) renamed /sheet5EFA929F/sheet5EF2B77E/SIGNAL
- net Net-(R25-Pad2) renamed /sheet5EFA929F/sheet5EF2B800/SIGNAL
- net Net-(R27-Pad2) renamed /sheet5EFA929F/sheet5EF2B8A4/SIGNAL
- net Net-(R29-Pad2) renamed /sheet5EFA929F/sheet5EF2B938/SIGNAL
- net Net-(R3-Pad2) renamed /Sheet595Neon/sheet5EF2B64C/SIGNAL
- net Net-(R31-Pad2) renamed /sheet5EFA929F/sheet5EF2B9F4/SIGNAL
- net Net-(R33-Pad2) renamed /sheet5EFA93E5/SheetSingleBulb/SIGNAL
- net Net-(R35-Pad2) renamed /sheet5EFA93E5/sheet5EF2B64C/SIGNAL
- net Net-(R37-Pad2) renamed /sheet5EFA93E5/sheet5EF2B6E0/SIGNAL
- net Net-(R39-Pad2) renamed /sheet5EFA93E5/sheet5EF2B77E/SIGNAL
- net Net-(R41-Pad2) renamed /sheet5EFA93E5/sheet5EF2B800/SIGNAL
- net Net-(R43-Pad2) renamed /sheet5EFA93E5/sheet5EF2B8A4/SIGNAL
- net Net-(R45-Pad2) renamed /sheet5EFA93E5/sheet5EF2B938/SIGNAL
- net Net-(R47-Pad2) renamed /sheet5EFA93E5/sheet5EF2B9F4/SIGNAL
- net Net-(R49-Pad2) renamed /sheet5EFA9519/SheetSingleBulb/SIGNAL
- net Net-(R5-Pad2) renamed /Sheet595Neon/sheet5EF2B6E0/SIGNAL
- net Net-(R51-Pad2) renamed /sheet5EFA9519/sheet5EF2B64C/SIGNAL
- net Net-(R53-Pad2) renamed /sheet5EFA9519/sheet5EF2B6E0/SIGNAL
- net Net-(R55-Pad2) renamed /sheet5EFA9519/sheet5EF2B77E/SIGNAL
- net Net-(R57-Pad2) renamed /sheet5EFA9519/sheet5EF2B800/SIGNAL
- net Net-(R59-Pad2) renamed /sheet5EFA9519/sheet5EF2B8A4/SIGNAL
- net Net-(R61-Pad2) renamed /sheet5EFA9519/sheet5EF2B938/SIGNAL
- net Net-(R63-Pad2) renamed /sheet5EFA9519/sheet5EF2B9F4/SIGNAL
- net Net-(R65-Pad2) renamed /sheet5EFAAFC3/SheetSingleBulb/SIGNAL
- net Net-(R67-Pad2) renamed /sheet5EFAAFC3/sheet5EF2B64C/SIGNAL
- net Net-(R69-Pad2) renamed /sheet5EFAAFC3/sheet5EF2B6E0/SIGNAL
- net Net-(R7-Pad2) renamed /Sheet595Neon/sheet5EF2B77E/SIGNAL
- net Net-(R71-Pad2) renamed /sheet5EFAAFC3/sheet5EF2B77E/SIGNAL
- net Net-(R73-Pad2) renamed /sheet5EFAAFC3/sheet5EF2B800/SIGNAL
- net Net-(R75-Pad2) renamed /sheet5EFAAFC3/sheet5EF2B8A4/SIGNAL
- net Net-(R77-Pad2) renamed /sheet5EFAAFC3/sheet5EF2B938/SIGNAL
- net Net-(R79-Pad2) renamed /sheet5EFAAFC3/sheet5EF2B9F4/SIGNAL
- net Net-(R81-Pad2) renamed /sheet5EFAAFC4/SheetSingleBulb/SIGNAL
- net Net-(R83-Pad2) renamed /sheet5EFAAFC4/sheet5EF2B64C/SIGNAL
- net Net-(R85-Pad2) renamed /sheet5EFAAFC4/sheet5EF2B6E0/SIGNAL
- net Net-(R87-Pad2) renamed /sheet5EFAAFC4/sheet5EF2B77E/SIGNAL
- net Net-(R89-Pad2) renamed /sheet5EFAAFC4/sheet5EF2B800/SIGNAL
- net Net-(R9-Pad2) renamed /Sheet595Neon/sheet5EF2B800/SIGNAL
- net Net-(R91-Pad2) renamed /sheet5EFAAFC4/sheet5EF2B8A4/SIGNAL
- net Net-(R93-Pad2) renamed /sheet5EFAAFC4/sheet5EF2B938/SIGNAL
- net Net-(R95-Pad2) renamed /sheet5EFAAFC4/sheet5EF2B9F4/SIGNAL
- net Net-(R97-Pad2) renamed /sheet5EFAAFC5/SheetSingleBulb/SIGNAL
- net Net-(R99-Pad2) renamed /sheet5EFAAFC5/sheet5EF2B64C/SIGNAL
Routing:
- net Net-(D3-Pad3): track 0.00 -> 4.50 mm
- net Net-(D8-Pad3): track 0.00 -> 4.50 mm
- net Net-(D7-Pad3): track 0.00 -> 4.50 mm
- net Net-(D6-Pad3): track 0.00 -> 4.50 mm
- net Net-(D2-Pad3): track 0.00 -> 4.50 mm
- net Net-(D53-Pad3): track 0.00 -> 4.50 mm
- net Net-(D21-Pad3): track 0.00 -> 4.50 mm
- net Net-(D16-Pad3): track 0.00 -> 4.50 mm
- net Net-(D32-Pad3): track 0.00 -> 4.50 mm
- net Net-(D26-Pad3): track 0.00 -> 4.50 mm
- net Net-(D60-Pad3): track 0.00 -> 4.50 mm
- net Net-(D56-Pad3): track 0.00 -> 4.50 mm
- net Net-(D30-Pad3): track 0.00 -> 4.50 mm
- net Net-(D58-Pad3): track 0.00 -> 4.50 mm
- net Net-(D52-Pad3): track 0.00 -> 4.50 mm
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Other:
- net class Default: clearance 0.2 -> 0.127; trace_width 0.25 -> 0.127; via_dia 0.8 -> 0.6; via_drill 0.4 -> 0.3
- rule trace_clearance: 0.2 -> 0.127
- rule trace_min: 0.2 -> 0.127
- rule via_min_size: 0.4 -> 0.6

Commit message: First row
Parts:
- removed D10, D11, D12, D13, D14, D15, D16, D17, D18, D19, D20, D21, D22, D23, D24, D25, D26, D27, D28, D29, D30, D31, D32, D33, D34, D35, D36, D37, D38, D39, D40, D41, D42, D43, D44, D45, D46, D47, D48, D49, D50, D51, D52, D53, D54, D55, D56, D57, D58, D59, D60, D61, D62, D63, D64, D9: Q_TRIAC_A1GA2, Package_TO_SOT_SMD:SOT-23
- removed NE10, NE11, NE12, NE13, NE14, NE15, NE16, NE17, NE18, NE19, NE20, NE21, NE22, NE23, NE24, NE25, NE26, NE27, NE28, NE29, NE30, NE31, NE32, NE33, NE34, NE35, NE36, NE37, NE38, NE39, NE40, NE41, NE42, NE43, NE44, NE45, NE46, NE47, NE48, NE49, NE50, NE51, NE52, NE53, NE54, NE55, NE56, NE57, NE58, NE59, NE60, NE61, NE62, NE63, NE64, NE9: Lamp_Neon, NeonMatrix_Connector:NeonBulb
- removed R100, R102, R104, R106, R108, R110, R112, R114, R116, R118, R120, R122, R124, R126, R128, R18, R20, R22, R24, R26, R28, R30, R32, R34, R36, R38, R40, R42, R44, R46, R48, R50, R52, R54, R56, R58, R60, R62, R64, R66, R68, R70, R72, R74, R76, R78, R80, R82, R84, R86, R88, R90, R92, R94, R96, R98: 33k, Resistor_SMD:R_0603_1608Metric
- removed R101, R103, R105, R107, R109, R111, R113, R115, R117, R119, R121, R123, R125, R127, R17, R19, R21, R23, R25, R27, R29, R31, R33, R35, R37, R39, R41, R43, R45, R47, R49, R51, R53, R55, R57, R59, R61, R63, R65, R67, R69, R71, R73, R75, R77, R79, R81, R83, R85, R87, R89, R91, R93, R95, R97, R99: 330k, Resistor_SMD:R_0402_1005Metric
- removed U2, U3, U4, U5, U6, U7, U8: 74HC595, Package_SO:SOIC-16_3.9x9.9mm_P1.27mm
- moved U1 4.33 mm to (43.6, 36.2)
Routing:
- net /Sheet595Neon/sheet5EF2B9F4/SIGNAL: track 0.00 -> 75.8 mm
- net /Sheet595Neon/sheet5EF2B938/SIGNAL: track 0.00 -> 66.8 mm
- net /Sheet595Neon/sheet5EF2B8A4/SIGNAL: track 0.00 -> 57.8 mm
- net /Sheet595Neon/sheet5EF2B800/SIGNAL: track 0.00 -> 49.4 mm
- net /Sheet595Neon/sheet5EF2B77E/SIGNAL: track 0.00 -> 40.9 mm
- net /Sheet595Neon/sheet5EF2B6E0/SIGNAL: track 0.00 -> 32.5 mm
- net /Sheet595Neon/sheet5EF2B64C/SIGNAL: track 0.00 -> 24.1 mm
- net /Sheet595Neon/SheetSingleBulb/SIGNAL: track 0.00 -> 21.2 mm
- net Net-(D53-Pad3): track 4.50 -> 0.00 mm
- net Net-(D21-Pad3): track 4.50 -> 0.00 mm
- net Net-(D16-Pad3): track 4.50 -> 0.00 mm
- net Net-(D32-Pad3): track 4.50 -> 0.00 mm
- net Net-(D26-Pad3): track 4.50 -> 0.00 mm
- net Net-(D60-Pad3): track 4.50 -> 0.00 mm
- net Net-(D56-Pad3): track 4.50 -> 0.00 mm
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
Commit message: First row
Parts:
- added D10: Q_TRIAC_A1GA2, Package_TO_SOT_SMD:SOT-23, F.Cu at (341.5, 89.5)
- added D11: Q_TRIAC_A1GA2, Package_TO_SOT_SMD:SOT-23, F.Cu at (295.7, 131.3)
- added D12: Q_TRIAC_A1GA2, Package_TO_SOT_SMD:SOT-23, F.Cu at (317.3, 116.4)
- added D13: Q_TRIAC_A1GA2, Package_TO_SOT_SMD:SOT-23, F.Cu at (411.4, 34.2)
- added D14: Q_TRIAC_A1GA2, Package_TO_SOT_SMD:SOT-23, F.Cu at (341.5, 103.0)
- added D15: Q_TRIAC_A1GA2, Package_TO_SOT_SMD:SOT-23, F.Cu at (363.1, 74.6)
- added D16: Q_TRIAC_A1GA2, Package_TO_SOT_SMD:SOT-23, F.Cu at (384.6, 61.1)
- added D17: Q_TRIAC_A1GA2, Package_TO_SOT_SMD:SOT-23, F.Cu at (317.3, 129.9)
- added D18: Q_TRIAC_A1GA2, Package_TO_SOT_SMD:SOT-23, F.Cu at (408.8, 47.7)
- added D19: Q_TRIAC_A1GA2, Package_TO_SOT_SMD:SOT-23, F.Cu at (363.1, 88.0)
- added D20: Q_TRIAC_A1GA2, Package_TO_SOT_SMD:SOT-23, F.Cu at (338.9, 116.4)
- added D21: Q_TRIAC_A1GA2, Package_TO_SOT_SMD:SOT-23, F.Cu at (363.1, 101.5)
- added D22: Q_TRIAC_A1GA2, Package_TO_SOT_SMD:SOT-23, F.Cu at (363.1, 61.1)
- added D23: Q_TRIAC_A1GA2, Package_TO_SOT_SMD:SOT-23, F.Cu at (406.2, 61.1)
- added D24: Q_TRIAC_A1GA2, Package_TO_SOT_SMD:SOT-23, F.Cu at (338.9, 129.9)
- added D25: Q_TRIAC_A1GA2, Package_TO_SOT_SMD:SOT-23, F.Cu at (430.4, 47.7)
- added D26: Q_TRIAC_A1GA2, Package_TO_SOT_SMD:SOT-23, F.Cu at (384.6, 88.0)
- added D27: Q_TRIAC_A1GA2, Package_TO_SOT_SMD:SOT-23, F.Cu at (363.1, 115.0)
- added D28: Q_TRIAC_A1GA2, Package_TO_SOT_SMD:SOT-23, F.Cu at (384.6, 101.5)
- added D29: Q_TRIAC_A1GA2, Package_TO_SOT_SMD:SOT-23, F.Cu at (406.2, 74.6)
- added D30: Q_TRIAC_A1GA2, Package_TO_SOT_SMD:SOT-23, F.Cu at (427.8, 61.1)
- added D31: Q_TRIAC_A1GA2, Package_TO_SOT_SMD:SOT-23, F.Cu at (360.5, 128.4)
- added D32: Q_TRIAC_A1GA2, Package_TO_SOT_SMD:SOT-23, F.Cu at (406.2, 88.0)
- added D33: Q_TRIAC_A1GA2, Package_TO_SOT_SMD:SOT-23, F.Cu at (384.6, 115.0)
- added D34: Q_TRIAC_A1GA2, Package_TO_SOT_SMD:SOT-23, F.Cu at (406.2, 101.5)
- added D35: Q_TRIAC_A1GA2, Package_TO_SOT_SMD:SOT-23, F.Cu at (427.8, 74.6)
- added D36: Q_TRIAC_A1GA2, Package_TO_SOT_SMD:SOT-23, F.Cu at (384.6, 74.6)
- added D37: Q_TRIAC_A1GA2, Package_TO_SOT_SMD:SOT-23, F.Cu at (300.9, 49.2)
- added D38: Q_TRIAC_A1GA2, Package_TO_SOT_SMD:SOT-23, F.Cu at (319.9, 62.6)
- added D39: Q_TRIAC_A1GA2, Package_TO_SOT_SMD:SOT-23, F.Cu at (298.3, 77.5)
- added D40: Q_TRIAC_A1GA2, Package_TO_SOT_SMD:SOT-23, F.Cu at (252.6, 120.8)
- added D41: Q_TRIAC_A1GA2, Package_TO_SOT_SMD:SOT-23, F.Cu at (346.6, 34.2)
- added D42: Q_TRIAC_A1GA2, Package_TO_SOT_SMD:SOT-23, F.Cu at (276.7, 91.0)
- added D43: Q_TRIAC_A1GA2, Package_TO_SOT_SMD:SOT-23, F.Cu at (322.5, 49.2)
- added D44: Q_TRIAC_A1GA2, Package_TO_SOT_SMD:SOT-23, F.Cu at (252.6, 107.3)
- added D45: Q_TRIAC_A1GA2, Package_TO_SOT_SMD:SOT-23, F.Cu at (298.3, 64.1)
- added D46: Q_TRIAC_A1GA2, Package_TO_SOT_SMD:SOT-23, F.Cu at (276.7, 77.5)
- added D47: Q_TRIAC_A1GA2, Package_TO_SOT_SMD:SOT-23, F.Cu at (325.0, 34.2)
- added D48: Q_TRIAC_A1GA2, Package_TO_SOT_SMD:SOT-23, F.Cu at (252.6, 93.9)
- added D49: Q_TRIAC_A1GA2, Package_TO_SOT_SMD:SOT-23, F.Cu at (276.7, 64.1)
- added D50: Q_TRIAC_A1GA2, Package_TO_SOT_SMD:SOT-23, F.Cu at (344.0, 47.7)
- added D51: Q_TRIAC_A1GA2, Package_TO_SOT_SMD:SOT-23, F.Cu at (274.2, 117.9)
- added D52: Q_TRIAC_A1GA2, Package_TO_SOT_SMD:SOT-23, F.Cu at (298.3, 91.0)
- added D53: Q_TRIAC_A1GA2, Package_TO_SOT_SMD:SOT-23, F.Cu at (368.2, 34.2)
- added D54: Q_TRIAC_A1GA2, Package_TO_SOT_SMD:SOT-23, F.Cu at (295.7, 104.4)
- added D55: Q_TRIAC_A1GA2, Package_TO_SOT_SMD:SOT-23, F.Cu at (319.9, 76.1)
- added D56: Q_TRIAC_A1GA2, Package_TO_SOT_SMD:SOT-23, F.Cu at (341.5, 62.6)
- added D57: Q_TRIAC_A1GA2, Package_TO_SOT_SMD:SOT-23, F.Cu at (365.6, 47.7)
- added D58: Q_TRIAC_A1GA2, Package_TO_SOT_SMD:SOT-23, F.Cu at (319.9, 89.5)
- added D59: Q_TRIAC_A1GA2, Package_TO_SOT_SMD:SOT-23, F.Cu at (274.2, 131.3)
- added D60: Q_TRIAC_A1GA2, Package_TO_SOT_SMD:SOT-23, F.Cu at (295.7, 117.9)
- added D61: Q_TRIAC_A1GA2, Package_TO_SOT_SMD:SOT-23, F.Cu at (389.8, 34.2)
- added D62: Q_TRIAC_A1GA2, Package_TO_SOT_SMD:SOT-23, F.Cu at (319.9, 103.0)
- added D63: Q_TRIAC_A1GA2, Package_TO_SOT_SMD:SOT-23, F.Cu at (341.5, 76.1)
- added D64: Q_TRIAC_A1GA2, Package_TO_SOT_SMD:SOT-23, F.Cu at (274.2, 104.4)
- added D9: Q_TRIAC_A1GA2, Package_TO_SOT_SMD:SOT-23, F.Cu at (387.2, 47.7)
- added NE10: Lamp_Neon, NeonMatrix_Connector:NeonBulb, F.Cu at (328.2, 89.6)
- added NE11: Lamp_Neon, NeonMatrix_Connector:NeonBulb, F.Cu at (282.4, 131.4)
- added NE12: Lamp_Neon, NeonMatrix_Connector:NeonBulb, F.Cu at (304.0, 116.5)
- added NE13: Lamp_Neon, NeonMatrix_Connector:NeonBulb, F.Cu at (398.1, 34.3)
- added NE14: Lamp_Neon, NeonMatrix_Connector:NeonBulb, F.Cu at (328.2, 103.0)
- added NE15: Lamp_Neon, NeonMatrix_Connector:NeonBulb, F.Cu at (349.8, 74.7)
- added NE16: Lamp_Neon, NeonMatrix_Connector:NeonBulb, F.Cu at (371.3, 61.2)
- added NE17: Lamp_Neon, NeonMatrix_Connector:NeonBulb, F.Cu at (304.0, 129.9)
- added NE18: Lamp_Neon, NeonMatrix_Connector:NeonBulb, F.Cu at (395.5, 47.8)
- added NE19: Lamp_Neon, NeonMatrix_Connector:NeonBulb, F.Cu at (349.8, 88.1)
- added NE20: Lamp_Neon, NeonMatrix_Connector:NeonBulb, F.Cu at (325.6, 116.5)
- added NE21: Lamp_Neon, NeonMatrix_Connector:NeonBulb, F.Cu at (349.8, 101.5)
- added NE22: Lamp_Neon, NeonMatrix_Connector:NeonBulb, F.Cu at (349.8, 61.2)
- added NE23: Lamp_Neon, NeonMatrix_Connector:NeonBulb, F.Cu at (392.9, 61.2)
- added NE24: Lamp_Neon, NeonMatrix_Connector:NeonBulb, F.Cu at (325.6, 129.9)
- added NE25: Lamp_Neon, NeonMatrix_Connector:NeonBulb, F.Cu at (417.1, 47.8)
- added NE26: Lamp_Neon, NeonMatrix_Connector:NeonBulb, F.Cu at (371.3, 88.1)
- added NE27: Lamp_Neon, NeonMatrix_Connector:NeonBulb, F.Cu at (349.8, 115.0)
- added NE28: Lamp_Neon, NeonMatrix_Connector:NeonBulb, F.Cu at (371.3, 101.5)
- added NE29: Lamp_Neon, NeonMatrix_Connector:NeonBulb, F.Cu at (392.9, 74.7)
- added NE30: Lamp_Neon, NeonMatrix_Connector:NeonBulb, F.Cu at (414.5, 61.2)
- added NE31: Lamp_Neon, NeonMatrix_Connector:NeonBulb, F.Cu at (347.2, 128.4)
- added NE32: Lamp_Neon, NeonMatrix_Connector:NeonBulb, F.Cu at (392.9, 88.1)
- added NE33: Lamp_Neon, NeonMatrix_Connector:NeonBulb, F.Cu at (371.3, 115.0)
- added NE34: Lamp_Neon, NeonMatrix_Connector:NeonBulb, F.Cu at (392.9, 101.5)
- added NE35: Lamp_Neon, NeonMatrix_Connector:NeonBulb, F.Cu at (414.5, 74.7)
- added NE36: Lamp_Neon, NeonMatrix_Connector:NeonBulb, F.Cu at (371.3, 74.7)
- added NE37: Lamp_Neon, NeonMatrix_Connector:NeonBulb, F.Cu at (287.6, 49.2)
- added NE38: Lamp_Neon, NeonMatrix_Connector:NeonBulb, F.Cu at (306.6, 62.7)
- added NE39: Lamp_Neon, NeonMatrix_Connector:NeonBulb, F.Cu at (285.0, 77.6)
- added NE40: Lamp_Neon, NeonMatrix_Connector:NeonBulb, F.Cu at (239.3, 120.8)
- added NE41: Lamp_Neon, NeonMatrix_Connector:NeonBulb, F.Cu at (333.3, 34.3)
- added NE42: Lamp_Neon, NeonMatrix_Connector:NeonBulb, F.Cu at (263.4, 91.0)
- added NE43: Lamp_Neon, NeonMatrix_Connector:NeonBulb, F.Cu at (309.2, 49.2)
- added NE44: Lamp_Neon, NeonMatrix_Connector:NeonBulb, F.Cu at (239.3, 107.4)
- added NE45: Lamp_Neon, NeonMatrix_Connector:NeonBulb, F.Cu at (285.0, 64.1)
- added NE46: Lamp_Neon, NeonMatrix_Connector:NeonBulb, F.Cu at (263.4, 77.6)
- added NE47: Lamp_Neon, NeonMatrix_Connector:NeonBulb, F.Cu at (311.7, 34.3)
- added NE48: Lamp_Neon, NeonMatrix_Connector:NeonBulb, F.Cu at (239.3, 93.9)
- added NE49: Lamp_Neon, NeonMatrix_Connector:NeonBulb, F.Cu at (263.4, 64.1)
- added NE50: Lamp_Neon, NeonMatrix_Connector:NeonBulb, F.Cu at (330.7, 47.8)
- added NE51: Lamp_Neon, NeonMatrix_Connector:NeonBulb, F.Cu at (260.9, 117.9)
- added NE52: Lamp_Neon, NeonMatrix_Connector:NeonBulb, F.Cu at (285.0, 91.0)
- added NE53: Lamp_Neon, NeonMatrix_Connector:NeonBulb, F.Cu at (354.9, 34.3)
- added NE54: Lamp_Neon, NeonMatrix_Connector:NeonBulb, F.Cu at (282.4, 104.5)
- added NE55: Lamp_Neon, NeonMatrix_Connector:NeonBulb, F.Cu at (306.6, 76.1)
- added NE56: Lamp_Neon, NeonMatrix_Connector:NeonBulb, F.Cu at (328.2, 62.7)
- added NE57: Lamp_Neon, NeonMatrix_Connector:NeonBulb, F.Cu at (352.3, 47.8)
- added NE58: Lamp_Neon, NeonMatrix_Connector:NeonBulb, F.Cu at (306.6, 89.6)
- added NE59: Lamp_Neon, NeonMatrix_Connector:NeonBulb, F.Cu at (260.9, 131.4)
- added NE60: Lamp_Neon, NeonMatrix_Connector:NeonBulb, F.Cu at (282.4, 117.9)
- added NE61: Lamp_Neon, NeonMatrix_Connector:NeonBulb, F.Cu at (376.5, 34.3)
- added NE62: Lamp_Neon, NeonMatrix_Connector:NeonBulb, F.Cu at (306.6, 103.0)
- added NE63: Lamp_Neon, NeonMatrix_Connector:NeonBulb, F.Cu at (328.2, 76.1)
- added NE64: Lamp_Neon, NeonMatrix_Connector:NeonBulb, F.Cu at (260.9, 104.5)
- added NE9: Lamp_Neon, NeonMatrix_Connector:NeonBulb, F.Cu at (373.9, 47.8)
- added R100: 33k, Resistor_SMD:R_0603_1608Metric, F.Cu at (330.4, 53.9)
- added R101: 330k, Resistor_SMD:R_0402_1005Metric, F.Cu at (273.4, 121.1)
- added R102: 33k, Resistor_SMD:R_0603_1608Metric, F.Cu at (260.5, 124.0)
- added R103: 330k, Resistor_SMD:R_0402_1005Metric, F.Cu at (297.5, 94.2)
- added R104: 33k, Resistor_SMD:R_0603_1608Metric, F.Cu at (284.7, 97.2)
- added R105: 330k, Resistor_SMD:R_0402_1005Metric, F.Cu at (367.4, 37.5)
- added R106: 33k, Resistor_SMD:R_0603_1608Metric, F.Cu at (354.6, 40.4)
- added R107: 330k, Resistor_SMD:R_0402_1005Metric, F.Cu at (295.0, 107.7)
- added R108: 33k, Resistor_SMD:R_0603_1608Metric, F.Cu at (282.1, 110.6)
- added R109: 330k, Resistor_SMD:R_0402_1005Metric, F.Cu at (319.1, 79.3)
- added R110: 33k, Resistor_SMD:R_0603_1608Metric, F.Cu at (306.3, 82.2)
- added R111: 330k, Resistor_SMD:R_0402_1005Metric, F.Cu at (340.7, 65.9)
- added R112: 33k, Resistor_SMD:R_0603_1608Metric, F.Cu at (327.9, 68.8)
- added R113: 330k, Resistor_SMD:R_0402_1005Metric, F.Cu at (364.9, 51.0)
- added R114: 33k, Resistor_SMD:R_0603_1608Metric, F.Cu at (352.0, 53.9)
- added R115: 330k, Resistor_SMD:R_0402_1005Metric, F.Cu at (319.1, 92.8)
- added R116: 33k, Resistor_SMD:R_0603_1608Metric, F.Cu at (306.3, 95.7)
- added R117: 330k, Resistor_SMD:R_0402_1005Metric, F.Cu at (273.4, 134.6)
- added R118: 33k, Resistor_SMD:R_0603_1608Metric, F.Cu at (260.5, 137.5)
- added R119: 330k, Resistor_SMD:R_0402_1005Metric, F.Cu at (295.0, 121.1)
- added R120: 33k, Resistor_SMD:R_0603_1608Metric, F.Cu at (282.1, 124.0)
- added R121: 330k, Resistor_SMD:R_0402_1005Metric, F.Cu at (389.0, 37.5)
- added R122: 33k, Resistor_SMD:R_0603_1608Metric, F.Cu at (376.1, 40.4)
- added R123: 330k, Resistor_SMD:R_0402_1005Metric, F.Cu at (319.1, 106.2)
- added R124: 33k, Resistor_SMD:R_0603_1608Metric, F.Cu at (306.3, 109.1)
- added R125: 330k, Resistor_SMD:R_0402_1005Metric, F.Cu at (340.7, 79.3)
- added R126: 33k, Resistor_SMD:R_0603_1608Metric, F.Cu at (327.9, 82.2)
- added R127: 330k, Resistor_SMD:R_0402_1005Metric, F.Cu at (273.4, 107.7)
- added R128: 33k, Resistor_SMD:R_0603_1608Metric, F.Cu at (260.5, 110.6)
- added R17: 330k, Resistor_SMD:R_0402_1005Metric, F.Cu at (386.4, 51.0)
- added R18: 33k, Resistor_SMD:R_0603_1608Metric, F.Cu at (373.6, 53.9)
- added R19: 330k, Resistor_SMD:R_0402_1005Metric, F.Cu at (340.7, 92.8)
- added R20: 33k, Resistor_SMD:R_0603_1608Metric, F.Cu at (327.9, 95.7)
- added R21: 330k, Resistor_SMD:R_0402_1005Metric, F.Cu at (295.0, 134.6)
- added R22: 33k, Resistor_SMD:R_0603_1608Metric, F.Cu at (282.1, 137.5)
- added R23: 330k, Resistor_SMD:R_0402_1005Metric, F.Cu at (316.6, 119.7)
- added R24: 33k, Resistor_SMD:R_0603_1608Metric, F.Cu at (303.7, 122.6)
- added R25: 330k, Resistor_SMD:R_0402_1005Metric, F.Cu at (410.6, 37.5)
- added R26: 33k, Resistor_SMD:R_0603_1608Metric, F.Cu at (397.7, 40.4)
- added R27: 330k, Resistor_SMD:R_0402_1005Metric, F.Cu at (340.7, 106.2)
- added R28: 33k, Resistor_SMD:R_0603_1608Metric, F.Cu at (327.9, 109.1)
- added R29: 330k, Resistor_SMD:R_0402_1005Metric, F.Cu at (362.3, 77.9)
- added R30: 33k, Resistor_SMD:R_0603_1608Metric, F.Cu at (349.4, 80.8)
- added R31: 330k, Resistor_SMD:R_0402_1005Metric, F.Cu at (383.9, 64.4)
- added R32: 33k, Resistor_SMD:R_0603_1608Metric, F.Cu at (371.0, 67.3)
- added R33: 330k, Resistor_SMD:R_0402_1005Metric, F.Cu at (316.6, 133.1)
- added R34: 33k, Resistor_SMD:R_0603_1608Metric, F.Cu at (303.7, 136.0)
- added R35: 330k, Resistor_SMD:R_0402_1005Metric, F.Cu at (408.0, 51.0)
- added R36: 33k, Resistor_SMD:R_0603_1608Metric, F.Cu at (395.2, 53.9)
- added R37: 330k, Resistor_SMD:R_0402_1005Metric, F.Cu at (362.3, 91.3)
- added R38: 33k, Resistor_SMD:R_0603_1608Metric, F.Cu at (349.4, 94.2)
- added R39: 330k, Resistor_SMD:R_0402_1005Metric, F.Cu at (338.1, 119.7)
- added R40: 33k, Resistor_SMD:R_0603_1608Metric, F.Cu at (325.3, 122.6)
- added R41: 330k, Resistor_SMD:R_0402_1005Metric, F.Cu at (362.3, 104.8)
- added R42: 33k, Resistor_SMD:R_0603_1608Metric, F.Cu at (349.4, 107.7)
- added R43: 330k, Resistor_SMD:R_0402_1005Metric, F.Cu at (362.3, 64.4)
- added R44: 33k, Resistor_SMD:R_0603_1608Metric, F.Cu at (349.4, 67.3)
- added R45: 330k, Resistor_SMD:R_0402_1005Metric, F.Cu at (405.4, 64.4)
- added R46: 33k, Resistor_SMD:R_0603_1608Metric, F.Cu at (392.6, 67.3)
- added R47: 330k, Resistor_SMD:R_0402_1005Metric, F.Cu at (338.1, 133.1)
- added R48: 33k, Resistor_SMD:R_0603_1608Metric, F.Cu at (325.3, 136.0)
- added R49: 330k, Resistor_SMD:R_0402_1005Metric, F.Cu at (429.6, 51.0)
- added R50: 33k, Resistor_SMD:R_0603_1608Metric, F.Cu at (416.7, 53.9)
- added R51: 330k, Resistor_SMD:R_0402_1005Metric, F.Cu at (383.9, 91.3)
- added R52: 33k, Resistor_SMD:R_0603_1608Metric, F.Cu at (371.0, 94.2)
- added R53: 330k, Resistor_SMD:R_0402_1005Metric, F.Cu at (362.3, 118.2)
- added R54: 33k, Resistor_SMD:R_0603_1608Metric, F.Cu at (349.4, 121.1)
- added R55: 330k, Resistor_SMD:R_0402_1005Metric, F.Cu at (383.9, 104.8)
- added R56: 33k, Resistor_SMD:R_0603_1608Metric, F.Cu at (371.0, 107.7)
- added R57: 330k, Resistor_SMD:R_0402_1005Metric, F.Cu at (405.4, 77.9)
- added R58: 33k, Resistor_SMD:R_0603_1608Metric, F.Cu at (392.6, 80.8)
- added R59: 330k, Resistor_SMD:R_0402_1005Metric, F.Cu at (427.0, 64.4)
- added R60: 33k, Resistor_SMD:R_0603_1608Metric, F.Cu at (414.2, 67.3)
- added R61: 330k, Resistor_SMD:R_0402_1005Metric, F.Cu at (359.7, 131.7)
- added R62: 33k, Resistor_SMD:R_0603_1608Metric, F.Cu at (346.9, 134.6)
- added R63: 330k, Resistor_SMD:R_0402_1005Metric, F.Cu at (405.4, 91.3)
- added R64: 33k, Resistor_SMD:R_0603_1608Metric, F.Cu at (392.6, 94.2)
- added R65: 330k, Resistor_SMD:R_0402_1005Metric, F.Cu at (383.9, 118.2)
- added R66: 33k, Resistor_SMD:R_0603_1608Metric, F.Cu at (371.0, 121.1)
- added R67: 330k, Resistor_SMD:R_0402_1005Metric, F.Cu at (405.4, 104.8)
- added R68: 33k, Resistor_SMD:R_0603_1608Metric, F.Cu at (392.6, 107.7)
- added R69: 330k, Resistor_SMD:R_0402_1005Metric, F.Cu at (427.0, 77.9)
- added R70: 33k, Resistor_SMD:R_0603_1608Metric, F.Cu at (414.2, 80.8)
- added R71: 330k, Resistor_SMD:R_0402_1005Metric, F.Cu at (383.9, 77.9)
- added R72: 33k, Resistor_SMD:R_0603_1608Metric, F.Cu at (371.0, 80.8)
- added R73: 330k, Resistor_SMD:R_0402_1005Metric, F.Cu at (300.1, 52.4)
- added R74: 33k, Resistor_SMD:R_0603_1608Metric, F.Cu at (287.3, 55.3)
- added R75: 330k, Resistor_SMD:R_0402_1005Metric, F.Cu at (319.1, 65.9)
- added R76: 33k, Resistor_SMD:R_0603_1608Metric, F.Cu at (306.3, 68.8)
- added R77: 330k, Resistor_SMD:R_0402_1005Metric, F.Cu at (297.5, 80.8)
- added R78: 33k, Resistor_SMD:R_0603_1608Metric, F.Cu at (284.7, 83.7)
- added R79: 330k, Resistor_SMD:R_0402_1005Metric, F.Cu at (251.8, 124.1)
- added R80: 33k, Resistor_SMD:R_0603_1608Metric, F.Cu at (239.0, 127.0)
- added R81: 330k, Resistor_SMD:R_0402_1005Metric, F.Cu at (345.8, 37.5)
- added R82: 33k, Resistor_SMD:R_0603_1608Metric, F.Cu at (333.0, 40.4)
- added R83: 330k, Resistor_SMD:R_0402_1005Metric, F.Cu at (276.0, 94.2)
- added R84: 33k, Resistor_SMD:R_0603_1608Metric, F.Cu at (263.1, 97.2)
- added R85: 330k, Resistor_SMD:R_0402_1005Metric, F.Cu at (321.7, 52.4)
- added R86: 33k, Resistor_SMD:R_0603_1608Metric, F.Cu at (308.8, 55.3)
- added R87: 330k, Resistor_SMD:R_0402_1005Metric, F.Cu at (251.8, 110.6)
- added R88: 33k, Resistor_SMD:R_0603_1608Metric, F.Cu at (239.0, 113.5)
- added R89: 330k, Resistor_SMD:R_0402_1005Metric, F.Cu at (297.5, 67.3)
- added R90: 33k, Resistor_SMD:R_0603_1608Metric, F.Cu at (284.7, 70.2)
- added R91: 330k, Resistor_SMD:R_0402_1005Metric, F.Cu at (276.0, 80.8)
- added R92: 33k, Resistor_SMD:R_0603_1608Metric, F.Cu at (263.1, 83.7)
- added R93: 330k, Resistor_SMD:R_0402_1005Metric, F.Cu at (324.3, 37.5)
- added R94: 33k, Resistor_SMD:R_0603_1608Metric, F.Cu at (311.4, 40.4)
- added R95: 330k, Resistor_SMD:R_0402_1005Metric, F.Cu at (251.8, 97.2)
- added R96: 33k, Resistor_SMD:R_0603_1608Metric, F.Cu at (239.0, 100.1)
- added R97: 330k, Resistor_SMD:R_0402_1005Metric, F.Cu at (276.0, 67.3)
- added R98: 33k, Resistor_SMD:R_0603_1608Metric, F.Cu at (263.1, 70.2)
- added R99: 330k, Resistor_SMD:R_0402_1005Metric, F.Cu at (343.3, 51.0)
- added U2: 74HC595, Package_SO:SOIC-16_3.9x9.9mm_P1.27mm, F.Cu at (28.0, 36.5)
- added U3: 74HC595, Package_SO:SOIC-16_3.9x9.9mm_P1.27mm, F.Cu at (28.0, 50.0)
- added U4: 74HC595, Package_SO:SOIC-16_3.9x9.9mm_P1.27mm, F.Cu at (28.0, 64.0)
- added U5: 74HC595, Package_SO:SOIC-16_3.9x9.9mm_P1.27mm, F.Cu at (28.0, 78.0)
- added U6: 74HC595, Package_SO:SOIC-16_3.9x9.9mm_P1.27mm, F.Cu at (28.0, 92.0)
- added U7: 74HC595, Package_SO:SOIC-16_3.9x9.9mm_P1.27mm, F.Cu at (28.0, 106.0)
- added U8: 74HC595, Package_SO:SOIC-16_3.9x9.9mm_P1.27mm, F.Cu at (28.0, 120.0)
- moved D7 20.4 mm to (92.7, 25.2)
- moved D4 20.4 mm to (66.4, 25.4)
- moved D8 20.4 mm to (101.5, 25.2)
- moved NE5 20.4 mm to (72.2, 28.2)
- moved NE6 20.4 mm to (80.9, 28.2)
- moved R14 20.4 mm to (91.0, 27.1)
- moved R16 20.4 mm to (99.7, 27.1)
- moved R8 20.4 mm to (64.6, 27.2)
- moved R9 20.4 mm to (77.4, 24.2)
- moved NE2 20.4 mm to (45.9, 28.2)
- moved D1 20.4 mm to (40.2, 25.3)
- moved D2 20.4 mm to (48.9, 25.3)
- moved D3 20.4 mm to (57.7, 25.3)
- moved D5 20.4 mm to (75.2, 25.2)
- moved D6 20.4 mm to (83.9, 25.3)
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
Commit message: First row
Parts:
- moved U3 1.70 mm to (28.0, 51.7)
- moved U4 1.70 mm to (28.0, 65.7)
- moved U5 1.70 mm to (28.0, 79.7)
- moved U6 1.70 mm to (28.0, 93.7)
- moved U7 1.70 mm to (28.0, 107.7)
- moved U8 1.70 mm to (28.0, 121.7)
- moved U2 0.90 mm to (28.0, 37.4)
Changed lines of the file:
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@@
   )
   (module Package_SO:SOIC-16_3.9x9.9mm_P1.27mm (layer F.Cu)
-    (at 28 120 180)
+    (at 28 121.7 180)
     (descr "SOIC, 16 Pin (JEDEC MS-012AC, https://www.analog.com/media/en/package-pcb-resources/package/pkg_pdf/soic_narrow-r/r_16.pdf), generated with kicad-footprint-generator ipc_gullwing_generator.py")
     (tags "SOIC SO")
@@
   )
   (module Package_SO:SOIC-16_3.9x9.9mm_P1.27mm (layer F.Cu)
-    (at 28 106 180)
+    (at 28 107.7 180)
     (descr "SOIC, 16 Pin (JEDEC MS-012AC, https://www.analog.com/media/en/package-pcb-resources/package/pkg_pdf/soic_narrow-r/r_16.pdf), generated with kicad-footprint-generator ipc_gullwing_generator.py")
     (tags "SOIC SO")
@@
   )
   (module Package_SO:SOIC-16_3.9x9.9mm_P1.27mm (layer F.Cu)
-    (at 28 92 180)
+    (at 28 93.7 180)
     (descr "SOIC, 16 Pin (JEDEC MS-012AC, https://www.analog.com/media/en/package-pcb-resources/package/pkg_pdf/soic_narrow-r/r_16.pdf), generated with kicad-footprint-generator ipc_gullwing_generator.py")
     (tags "SOIC SO")
@@
   )
   (module Package_SO:SOIC-16_3.9x9.9mm_P1.27mm (layer F.Cu)
-    (at 28 78 180)
+    (at 28 79.7 180)
     (descr "SOIC, 16 Pin (JEDEC MS-012AC, https://www.analog.com/media/en/package-pcb-resources/package/pkg_pdf/soic_narrow-r/r_16.pdf), generated with kicad-footprint-generator ipc_gullwing_generator.py")
     (tags "SOIC SO")
@@
   )
   (module Package_SO:SOIC-16_3.9x9.9mm_P1.27mm (layer F.Cu)
-    (at 28 64 180)
+    (at 28 65.7 180)
     (descr "SOIC, 16 Pin (JEDEC MS-012AC, https://www.analog.com/media/en/package-pcb-resources/package/pkg_pdf/soic_narrow-r/r_16.pdf), generated with kicad-footprint-generator ipc_gullwing_generator.py")
     (tags "SOIC SO")
@@
   )
   (module Package_SO:SOIC-16_3.9x9.9mm_P1.27mm (layer F.Cu)
-    (at 28 50 180)
+    (at 28 51.7 180)
     (descr "SOIC, 16 Pin (JEDEC MS-012AC, https://www.analog.com/media/en/package-pcb-resources/package/pkg_pdf/soic_narrow-r/r_16.pdf), generated with kicad-footprint-generator ipc_gullwing_generator.py")
     (tags "SOIC SO")
@@
   )
   (module Package_SO:SOIC-16_3.9x9.9mm_P1.27mm (layer F.Cu)
-    (at 28 36.5 180)
-    (descr "SOIC, 16 Pin (JEDEC MS-012AC, https://www.analog.com/media/en/package-pcb-resources/package/pkg_pdf/soic_narrow-r/r_16.pdf), generated with kicad-footprint-generator ipc_gullwing_generator.py")
-    (tags "SOIC SO")
+    (at 28 37.4 180)
+    (descr "SOIC, 16 Pin (JEDEC MS-012AC, https://www.analog.com/media/en/package-pcb-resources/package/pkg_pdf/soic_narrow-r/r_16.pdf), generated with kicad-footprint-generator ipc_gullwing_generator.py")
+    (tags "SOIC SO")

Commit message: First row
Parts:
- removed D10, D11, D12, D13, D14, D15, D16, D17, D18, D19, D20, D21, D22, D23, D24, D25, D26, D27, D28, D29, D30, D31, D32, D33, D34, D35, D36, D37, D38, D39, D40, D41, D42, D43, D44, D45, D46, D47, D48, D49, D50, D51, D52, D53, D54, D55, D56, D57, D58, D59, D60, D61, D62, D63, D64, D9: Q_TRIAC_A1GA2, Package_TO_SOT_SMD:SOT-23
- removed NE10, NE11, NE12, NE13, NE14, NE15, NE16, NE17, NE18, NE19, NE20, NE21, NE22, NE23, NE24, NE25, NE26, NE27, NE28, NE29, NE30, NE31, NE32, NE33, NE34, NE35, NE36, NE37, NE38, NE39, NE40, NE41, NE42, NE43, NE44, NE45, NE46, NE47, NE48, NE49, NE50, NE51, NE52, NE53, NE54, NE55, NE56, NE57, NE58, NE59, NE60, NE61, NE62, NE63, NE64, NE9: Lamp_Neon, NeonMatrix_Connector:NeonBulb
- removed R100, R102, R104, R106, R108, R110, R112, R114, R116, R118, R120, R122, R124, R126, R128, R18, R20, R22, R24, R26, R28, R30, R32, R34, R36, R38, R40, R42, R44, R46, R48, R50, R52, R54, R56, R58, R60, R62, R64, R66, R68, R70, R72, R74, R76, R78, R80, R82, R84, R86, R88, R90, R92, R94, R96, R98: 33k, Resistor_SMD:R_0603_1608Metric
- removed R101, R103, R105, R107, R109, R111, R113, R115, R117, R119, R121, R123, R125, R127, R17, R19, R21, R23, R25, R27, R29, R31, R33, R35, R37, R39, R41, R43, R45, R47, R49, R51, R53, R55, R57, R59, R61, R63, R65, R67, R69, R71, R73, R75, R77, R79, R81, R83, R85, R87, R89, R91, R93, R95, R97, R99: 330k, Resistor_SMD:R_0402_1005Metric
Routing:
- net LINE: track 0.00 -> 104.4 mm
- net GND: track 0.00 -> 9.23 mm, vias 0 -> 9
- added copper zone on B.Cu, net GND
Other:
- board outline added: 86 x 116 mm
- net class HV added: clearance 0.5, trace_width 0.127, via_dia 0.6, via_drill 0.3
