File: NeonMatrix.sch (KiCad schematic (older format))
At the start: 14 parts, among them J1 Mains, J2 Data, M1 B0505S, U10 ADuM1200AR, U9 ADuM1200AR

Commit message: RevA, Add production files
Parts:
- added C15, C16: 100n, Capacitor_SMD:C_0805_2012Metric, symbol Device:C
- added U11: ADuM1200AR, Package_SO:SOIC-8_3.9x4.9mm_P1.27mm, symbol Isolator:ADuM1200AR
- J2: footprint Connector_PinHeader_2.54mm:PinHeader_1x06_P2.54mm_Vertical -> Connector_PinHeader_2.54mm:PinHeader_1x07_P2.54mm_Vertical; symbol Connector:Conn_01x06_Male -> Connector:Conn_01x07_Male
Connections:
- net +3V3: now also C16.1, U11.1 (VDD1)
- net GND: now also C16.2, U11.3 (VIB), U11.4 (GND1)
- net ISO_5V: now also C15.1, U11.8 (VDD2)
- net ISO_GND: now also C15.2, U11.5 (GND2)
- new net DATAOUT: U11.2 (VIA)
- new net ISO_DATAOUT: J2.7 (Pin_7), U11.7 (VOA)
Other:
- moved on the sheet: C2, C3, C4, C5, M1, TP1, TP2, U10, U9
